File: kicad/proto_ads_bee_mcu_board/proto_ads_bee_mcu_board.kicad_sch (KiCad schematic)
At the start: 29 parts, among them J1 Conn_ARM_JTAG_SWD_10, J2 Conn_01x03_Pin, J3 Conn_01x02_Pin, J4 Conn_01x04_Pin, J5 Conn_01x02_Pin, Q1 2N7002, U1 Pico, U2 MCP6541

Commit message: Move pins to setup decode blanking
Parts:
- removed U2: MCP6541, Package_TO_SOT_SMD:SOT-23-5, symbol Custom_Comparator:MCP6541
- added R8: 1k, symbol Device:R_US
- added U3: LMV331, symbol Comparator:LMV331
Connections:
- net +3V3: now also R8.1, U3.5 (V+)
- net COMP_REF: now also U3.1 (+)
- net COMP_SIG: now also U3.3 (-)
- net GND: now also U3.2 (V-)
- net PULSES: now reaches U1.25 (GPIO19)
- net PULSES: now also J5.1 (Pin_1), R8.2, U3.4
- net DECODE: now reaches U1.26 (GPIO20)
- net DECODE: now also U1.27 (GPIO21)
- net COMP_OUT: no longer names the net of U1.34 (GPIO28_ADC2)
- net COMP_OUT: no longer J5.1 (Pin_1)
- no-connect marks 29 -> 27
Other:
- moved on the sheet: J5
