File: kicad/adsbee_1090/adsbee_1090.kicad_pcb (KiCad board)
At the start: 6 copper layers, 45 x 30 mm, 108 parts, among them J1 U.FL 6GHz 50R, J2 USB_C_Receptacle_USB2.0_16P, J3 Conn_02x03_Pin, J4 Conn_ARM_JTAG_SWD_10, J5 Conn_01x05_Pin, J6 Conn_01x11_Pin, SW1 SN74LVC1G3157, SW2 SN74LVC1G3157, SW3 SW_Push, SW4 SW_Push, U1 BGA2818, U10 AMS1117-3.3, U2 AD8313xRM, U3 TLV3542, U4 MCP4017-104E 100k, U5 MCP6566, U6 M24C02-RDW, U7 W25Q128JVS, U8 RP2040, U9 ESP32-PICO-MINI-02U, X1 SF2321D, Y1 12.000MHz 18pF ±20ppm 80R

Commit message: Mega commit
Fix decoding for 56-bit squitter packets

Add MESSAGE_INTERVAL delimiter to MAVLINK reporting

Add MAVLINK1 support and 3d printed parts.

* Add support for MAVLINK1 to enable use in legacy PingRX projects.
* Rename MAVLINK protocol to MAVLINK2.
* Add 3D printed parts for solar feeder enclosure.
* Add PCB mounting hole dimensions to PCB design file.

Re-release Rev C manufacturing files, ESP docker

Add ESP32 project and add WiFi AT command to Pico
Other:
- board text added: "0.1500 mm / 0.1500 mm"
- board text added: "ALL 0.3MM VIAS TO BE EPOXY FILLED AND CAPPED WITH COPPER."
- board text added: "NOTES: UNLESS OTHERWISE SPECIFIED. 1. MATERIAL: A. FR4 Tg 150 C OR EQUIVALENT. B. EQUIVALENT MATERIAL SHALL BE RoHS COMPLIANT, HALOGEN FREE AND APPROVED BY PANTS FOR BIRDS LLC. C. THICKNESS OF INDIVIDUAL COPPER CLAD SHEETS SHALL BE IN AS DEFINED IN STACK-UP. 2. ETCH GEOMETRY: A. MEASURE WIDTH FROM THE BASE OF THE METALIZATION. B. MINIMUM LINE WIDTH: 0.15 MM OUTER, 0.15 MM INNER LAYERS. C. FINISHE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"
- board text added: "Yes"
- board text removed: "0.0000 mm / 0.0000 mm"

Commit message: Add Rev D PCBA files
Parts:
- removed C7, C8: 39pF, Capacitor_SMD:C_0402_1005Metric
- removed U1: BGA2818, Package_TO_SOT_SMD:SOT-363_SC-70-6
- added C33: 22nF, Capacitor_SMD:C_0402_1005Metric, F.Cu at (58.2, 42.6)
- added C34: 10uF, Capacitor_SMD:C_0805_2012Metric, F.Cu at (67.4, 57.5)
- added C35: 100pF, Capacitor_SMD:C_0402_1005Metric, F.Cu at (71.0, 45.6)
- added C36: 100pF, Capacitor_SMD:C_0402_1005Metric, F.Cu at (69.9, 51.1)
- added C37: 12pF, Capacitor_SMD:C_0402_1005Metric, F.Cu at (73.4, 44.1)
- added C38: 12pF, Capacitor_SMD:C_0402_1005Metric, F.Cu at (71.5, 50.5)
- added C39: 0.1uF, Capacitor_SMD:C_0402_1005Metric, F.Cu at (73.0, 49.3)
- added D7: ORANGE, LED_SMD:LED_0603_1608Metric, F.Cu at (46.5, 43.0)
- added L2: 27nH RF, Inductor_SMD:L_0402_1005Metric, F.Cu at (73.0, 45.6)
- added L3: 82nH RF, Inductor_SMD:L_0402_1005Metric, F.Cu at (69.9, 50.1)
- added R28: 1k, Resistor_SMD:R_0402_1005Metric, F.Cu at (61.8, 58.7)
- added R29: 20R, Resistor_SMD:R_0402_1005Metric, F.Cu at (66.9, 48.8)
- added R30: 750R, Resistor_SMD:R_0402_1005Metric, F.Cu at (49.4, 40.8)
- added R31: 6.8k, Resistor_SMD:R_0402_1005Metric, F.Cu at (73.0, 47.3)
- added R32: 0R, Resistor_SMD:R_0402_1005Metric, F.Cu at (68.4, 49.6)
- added U11: BLB01, Custom_Package_DFN_QFN:DFN-8-1EP_2x2mm_P0.5mm_EP0.9x1.5mm, F.Cu at (71.2, 47.9)
- C2: value 22nF -> 100pF
- J5: value Conn_01x05_Pin -> 1x5 2.54mm Pin Header
- J6: value Conn_01x11_Pin -> 1x11 2.54mm Pin Header
- X1: value SF2321D -> TA2003A; footprint Custom_Filter:Filter_SAW-6_3.8x3.8mm -> Custom_Filter:Filter_SAW-6_3.0x3.0mm
- moved C2 10.2 mm to (72.0, 40.1), turned to -90 degrees
- moved X1 1.41 mm to (70.5, 43.1)
- moved TP2 1.12 mm to (71.6, 48.8)
- moved C19 0.83 mm to (50.5, 40.8)
- moved TP8 0.42 mm to (58.1, 43.6)
- moved C10 0.36 mm to (70.5, 52.6)
- moved C3 0.36 mm to (72.5, 53.6)
- moved C4 0.36 mm to (69.5, 53.6)
- moved C9 0.36 mm to (71.5, 52.6)
- moved L1 0.36 mm to (71.0, 54.1)
- moved R2 0.28 mm to (73.4, 55.5)
- moved R3 0.28 mm to (68.6, 55.5)
- moved PCB1 0.21 mm to (76.7, 46.1)
- moved R5 0.20 mm to (72.0, 61.7)
- moved U2 0.20 mm to (71.0, 57.8)
Connections:
- net /MTL_BIAS renamed /TL_BIAS
- net /MTL_HI_BIAS renamed /TL_LO_BIAS
- net /MTL_HI_PWM renamed /TL_LO_PWM
- net /MTL_LO_BIAS renamed /TL_HI_BIAS
- net /MTL_LO_PWM renamed /TL_HI_PWM
- C2 pad 1: +3V3 -> /RF_IN
- C2 pad 2: GND -> /RF_SAW_IN
- C9 pad 1: Net-(C9-Pad1) -> /RF_LNA_OUT
- SW2 pad 1: /RSSI_PEAK -> Net-(SW2-B2)
- U3 pad 3: /RF_DET_OUT -> /RF_DET_OUT_FILT
- U9 pad 29: unconnected-(U9-GPIO5-Pad29) -> /ESP_LED
Routing:
- net /ESP_LED: track 0.00 -> 15.9 mm, vias 0 -> 2
- net Net-(SW2-B2): track 0.00 -> 8.23 mm, vias 0 -> 2
- net /RF_DET_OUT: track 13.2 -> 7.01 mm
- net /RF_DET_OUT_FILT: track 0.00 -> 5.86 mm
- net /RSSI_PEAK: track 12.0 -> 6.21 mm, vias 2 -> 0
- net /GNSS_PPS: track 28.6 -> 33.1 mm, vias 1 -> 2
- net Net-(U11-Vcc): track 0.00 -> 3.50 mm
- net Net-(D7-K): track 0.00 -> 2.81 mm
- net /RF_LNA_OUT': track 0.00 -> 2.27 mm
- net /~{RESET}: track 18.2 -> 20.4 mm
- net Net-(C35-Pad2): track 0.00 -> 2.10 mm
- net Net-(C36-Pad1): track 0.00 -> 2.02 mm
- net /RF_LEVEL: track 18.1 -> 16.2 mm, vias 3 -> 4
- net /RF_IN: track 4.42 -> 2.59 mm
- net Net-(C9-Pad1): track 1.27 -> 0.00 mm
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- added copper zone on In3.Cu, net GND
- removed copper zone on In4.Cu, net GND
Other:
- board text added: "NET"
- board text added: "TL_BIAS"
- board text added: "TL_HI_BIAS"
- board text added: "TL_LO_BIAS"
- board text removed: "MTL_BIAS"
- board text removed: "MTL_HI_BIAS"
- board text removed: "MTL_LO_BIAS"

Commit message: Update Rev D fab files
Parts:
- renumbered C39 to C1, C35 to C10, C38 to C11, C10 to C12, C31 to C14, C32 to C15, C1 to C16, C5 to C17, C11 to C18, C12 to C19, C6 to C2, C16 to C20, C17 to C21, C18 to C22, C19 to C23, C20 to C24, C21 to C25, C22 to C26, C23 to C27, C24 to C28, C25 to C29, C26 to C30, C14 to C31, C27 to C32, C15 to C33, C28 to C34, C29 to C35, C33 to C36, C30 to C37, C37 to C5, C36 to C6, C9 to C7, C34 to C8, C2 to C9, D3 to D2, D4 to D3, D5 to D4, D7 to D5, D2 to D6, D6 to D7, J6 to J5, J5 to J6, L2 to L1, L3 to L2, L1 to L3, R2 to R1, R9 to R10, R10 to R11, R6 to R12, R26 to R13, R27 to R14, R30 to R15, R11 to R16, R12 to R17, R13 to R18, R14 to R19, R3 to R2, R15 to R20, R16 to R21, R17 to R22, R29 to R23, R21 to R24, R8 to R25, R24 to R26, R25 to R27, R18 to R28, R19 to R29, R31 to R3, R20 to R30, R22 to R31, R23 to R32, R32 to R4, R28 to R5, R5 to R6, R1 to R8, R4 to R9, TP3 to TP1, TP6 to TP2, TP7 to TP3, TP1 to TP4, TP2 to TP5, TP4 to TP6, TP5 to TP7, U3 to U1, U9 to U10, U11 to U2, U2 to U3, U10 to U5, U5 to U6, U6 to U7, U7 to U8, U8 to U9
