File: kicad/adsbee_1090/adsbee_1090.kicad_sch (KiCad schematic)
At the start: 84 parts, among them J1 U.FL 6GHz 50R, J2 USB_Micro-B_Receptacle, J3 Conn_02x03_Odd_Even, J4 Conn_ARM_JTAG_SWD_10, Q1 BSS84, SW1 SW_Push, SW2 SW_Push, SW3 SN74LVC1G3157, U1 AD8314, U2 BGA2818, U3 MCP6566, U4 AP2112K-3.3, U5 W25Q128JVS, U6 RP2040, U7 OPA358AIDCKR, X1 SF2321D, Y1 12.000MHz 18pF ±20ppm 80R

Commit message: Make ADSBee PCBA Rev C
* production folder for JLCPCB has U5 and X1 removed due to stockout.
Parts:
- removed C1: 0.1uF, Capacitor_SMD:C_0402_1005Metric, symbol Device:C
- removed C21: 1uF, Capacitor_SMD:C_0603_1608Metric, symbol Device:C
- removed C27, C8: DNP, Capacitor_SMD:C_0402_1005Metric, symbol Device:C
- removed J2: USB_Micro-B_Receptacle, Custom_Connector_USB:USB_Micro-B_Amphenol_10118193-0001LF_Horizontal, symbol Connector:USB_B_Micro
- removed L2: 12nH, Inductor_SMD:L_0402_1005Metric, symbol Device:L
- removed Q1: BSS84, Package_TO_SOT_SMD:SOT-23, symbol Transistor_FET:BSS84
- removed R13: 10k, Resistor_SMD:R_0402_1005Metric, symbol Device:R_US
- removed R6: 115R, Resistor_SMD:R_0402_1005Metric, symbol Device:R_US
- removed U1: AD8314, Custom_Package_CSP:LFCSP-8-1EP_3x2mm_P0.5mm_EP1.6x1.65mm, symbol Custom_RF_Amplifier:AD8314
- removed U4: AP2112K-3.3, Package_TO_SOT_SMD:SOT-23-5, symbol Regulator_Linear:AP2112K-3.3
- removed U7: OPA358AIDCKR, Package_TO_SOT_SMD:SOT-363_SC-70-6, symbol Custom_Amplifier_Operational:OPA358AIDCKR
- added C10, C9: 3pF, Capacitor_SMD:C_0402_1005Metric, symbol Device:C
- added C13, C14, C4, C6: 0.1uF, Capacitor_SMD:C_0402_1005Metric, symbol Device:C
- added C32: 10uF, Capacitor_SMD:C_0805_2012Metric, symbol Device:C
- added D6: 20V 1A, Diode_SMD:D_SOD-123, symbol Device:D_Schottky
- added F1, F2: 6V 200mA, Fuse:Fuse_0402_1005Metric, symbol Device:Polyfuse
- added J2: USB_C_Receptacle_USB2.0_16P, Custom_Connector_USB:USB_C_Receptacle_GCT_USB4105-xx-A_16P_TopMnt_Horizontal, symbol Connector:USB_C_Receptacle_USB2.0_16P
- added J5: Conn_01x05_Pin, Connector_PinHeader_2.54mm:PinHeader_1x05_P2.54mm_Vertical, symbol Connector:Conn_01x05_Pin
- added J6: Conn_01x11_Pin, Connector_PinHeader_2.54mm:PinHeader_1x11_P2.54mm_Vertical, symbol Connector:Conn_01x11_Pin
- added R10, R9: 5.1k, Resistor_SMD:R_0402_1005Metric, symbol Device:R_US
- added R11, R12, R16, R17: 2.2k, Resistor_SMD:R_0402_1005Metric, symbol Device:R_US
- added R18, R19, R20: 0R, Resistor_SMD:R_0402_1005Metric, symbol Device:R_US
- added R2: 10R, Resistor_SMD:R_0402_1005Metric, symbol Device:R_US
- added R22, R23: 10k, Resistor_SMD:R_0402_1005Metric, symbol Device:R_US
- added R8: 20R, Resistor_SMD:R_0402_1005Metric, symbol Device:R_US
- added SW2: SN74LVC1G3157, Package_TO_SOT_SMD:SOT-363_SC-70-6, symbol Custom_Analog_Switch:SN74LVC1G3157
- added TP3, TP6, TP7: TestPoint, TestPoint:TestPoint_Pad_D1.0mm, symbol Connector:TestPoint
- added U10: AMS1117-3.3, Package_TO_SOT_SMD:SOT-223-3_TabPin2, symbol Regulator_Linear:AMS1117-3.3
- added U2: AD8313xRM, Package_SO:MSOP-8_3x3mm_P0.65mm, symbol RF_Amplifier:AD8313xRM
- added U3: TLV3542, Package_SO:VSSOP-8_3.0x3.0mm_P0.65mm, symbol Custom_Amplifier_Operational:TLV3542
- added U4: MCP4017-104E 100k, Package_TO_SOT_SMD:SOT-363_SC-70-6, symbol Potentiometer_Digital:MCP4017-xxxxLT
- added U6: M24C02-RDW, Package_SO:TSSOP-8_4.4x3mm_P0.65mm, symbol Memory_EEPROM:M24C02-RDW
- added U9: ESP32-PICO-MINI-02U, Custom_MCU_Espressif:ESP32-PICO-MINI-02U, symbol Custom_MCU_Espressif:ESP32-PICO-MINI-02
- C1, C2, C3: MPN CC0402KRX7R7BB104 -> C60474; OEM PN (none) -> CC0402KRX7R7BB104
- C15: renamed from C29; MPN CC0402KRX7R9BB223 -> C107026; OEM PN (none) -> CC0402KRX7R9BB223
- C16: renamed from C10; MPN CC0402KRX7R7BB104 -> C60474; OEM PN (none) -> CC0402KRX7R7BB104
- C17: renamed from C11; MPN CC0402KRX7R7BB104 -> C60474; OEM PN (none) -> CC0402KRX7R7BB104
- C18: renamed from C12; MPN CC0402KRX7R7BB104 -> C60474; OEM PN (none) -> CC0402KRX7R7BB104
- C19: renamed from C13; MPN CC0402KRX7R7BB104 -> C60474; OEM PN (none) -> CC0402KRX7R7BB104
- C2: renamed from C1; MPN CC0402KRX7R9BB223 -> C107026; OEM PN (none) -> CC0402KRX7R9BB223
- C20: renamed from C14; MPN CC0402KRX7R7BB104 -> C60474; OEM PN (none) -> CC0402KRX7R7BB104
- C21: renamed from C15; MPN CC0402KRX7R7BB104 -> C60474; OEM PN (none) -> CC0402KRX7R7BB104
- C22: renamed from C16; MPN CC0402KRX7R7BB104 -> C60474; OEM PN (none) -> CC0402KRX7R7BB104
- C23: renamed from C17; MPN CC0402KRX7R7BB104 -> C60474; OEM PN (none) -> CC0402KRX7R7BB104
- C24: renamed from C18; MPN CL10B105KA8NNNC -> C29936; OEM PN (none) -> CL10B105KA8NNNC
- C25: renamed from C19; MPN CL10B105KA8NNNC -> C29936; OEM PN (none) -> CL10B105KA8NNNC
- C26: value 7pF -> 0.1uF; MPN CC0402CRNPO9BN7R0 -> C60474; OEM PN (none) -> CC0402KRX7R7BB104
- C27: renamed from C20; MPN CC0402KRX7R7BB104 -> C60474; OEM PN (none) -> CC0402KRX7R7BB104
- C28: renamed from C23; MPN CC0402JRNPO9BN270 -> C107002; OEM PN (none) -> CC0402JRNPO9BN270
- C29: renamed from C24; MPN CC0402JRNPO9BN270 -> C107002; OEM PN (none) -> CC0402JRNPO9BN270
- C30: renamed from C25; MPN CC0402KRX7R7BB104 -> C60474; OEM PN (none) -> CC0402KRX7R7BB104
- C31: renamed from C22; value 1uF -> 10uF; footprint Capacitor_SMD:C_0603_1608Metric -> Capacitor_SMD:C_0805_2012Metric; MPN CL10B105KA8NNNC -> C95841; OEM PN (none) -> CL21B106KOQNNNE; Standard Cost 0.01 -> 0.02
- C7: renamed from C5; MPN CC0402JRNPO9BN390 -> C106223; OEM PN (none) -> CC0402JRNPO9BN390
- C8: renamed from C6; MPN CC0402JRNPO9BN390 -> C106223; OEM PN (none) -> CC0402JRNPO9BN390
- CR1: MPN DRTR5V0U2SR-7 -> C443828; Note (none) -> Low LCSC stock.; OEM PN (none) -> DRTR5V0U2SR-7
- D1: MPN ESD7351XV2T1G -> C2912559; Note (none) -> Substituted with TECH PUBLIC dupe due to no stock of onsemi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; OEM PN (none) -> ESD7351XV2T1G
- D2: renamed from D5; MPN PMEG2010ER,115 -> C82288; OEM PN (none) -> PMEG2010ER,115; Standard Cost 0.11 -> 0.06
- D3: renamed from D2; MPN PMEG2010ER,115 -> C82288; OEM PN (none) -> PMEG2010ER,115; Standard Cost 0.11 -> 0.06
- D4: renamed from D3; MPN SML-D12U8WT86 -> C510027; OEM PN (none) -> SML-D12U8WT86; Standard Cost 0.07 -> 0.04
- D5: renamed from D4; MPN SML-D12M8WT86 -> C510025; OEM PN (none) -> SML-D12M8WT86; Standard Cost 0.07 -> 0.04
- J1: MPN A-1JB -> C88374; Note (none) -> (80) suffix denotes reel size, can be substituted.; OEM PN (none) -> U.FL-R-SMT-1(80)
- J3: value Conn_02x03_Odd_Even -> Conn_02x03_Pin; footprint Connector_PinHeader_2.54mm:PinHeader_2x03_P2.54mm_Vertical -> Connector_PinHeader_1.27mm:PinHeader_2x03_P1.27mm_Vertical_SMD; MPN X6521WV-2x03H-C60D30 -> C3975186; OEM PN (none) -> PZ127-2-03-S; Standard Cost 0.06 -> 0.04
- J4: MPN 20021221-00010C4LF -> C2935458; Note (none) -> Couldn't find connector with keying for SWD connector.; OEM PN (none) -> PZ127VS-12-10-H10-A38; Standard Cost 0.67 -> 0.10
- L1: value 100nH -> 8.2nH RF; MPN LQG15HSR10J02D -> C361505; Note (none) -> Looking for a wire wound inductor with similar performance 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; OEM PN (none) -> SDWL1005C8N2JSTF; Standard Cost 0.04 -> 0.03
- PCB1: OEM PN (none) -> adsbee_1090; REV REV B -> REV C
- R1: renamed from R2; MPN RC0402FR-0710KL -> C60490; OEM PN (none) -> RC0402FR-0710KL
- R13: renamed from R10; MPN RC0402FR-0727R4L -> C284479; Note (none) -> Substituted with part from Viking Tech due to no LCSC stock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; OEM PN (none) -> RC0402FR-0727R4L
- R14: renamed from R11; MPN RC0402FR-0727R4L -> C284479; Note (none) -> Substituted with part from Viking Tech due to no LCSC stock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; OEM PN (none) -> RC0402FR-0727R4L
- R15: renamed from R12; MPN RC0402FR-0710KL -> C60490; OEM PN (none) -> RC0402FR-0710KL
- R21: renamed from R14; MPN RC0402FR-071KL -> C106235; OEM PN (none) -> RC0402FR-071KL
- R24: renamed from R15; MPN RC0402FR-071KL -> C106235; OEM PN (none) -> RC0402FR-071KL
- R25: renamed from R16; MPN RC0402FR-0710KL -> C60490; OEM PN (none) -> RC0402FR-0710KL
- R26: renamed from R8; MPN RC0402FR-07287RL -> C375493; OEM PN (none) -> RC0402FR-07287RL
- R27: renamed from R9; MPN RC0402FR-07115RL -> C295872; OEM PN (none) -> RC0402FR-07115RL
- R3: value 10k -> 10R; MPN RC0402FR-0710KL -> C138066; OEM PN (none) -> RC0402FR-0710RL
- R4: renamed from R1; MPN RC0402FR-0710KL -> C60490; OEM PN (none) -> RC0402FR-0710KL
- R5: value 10k -> 0R; MPN RC0402FR-0710KL -> C60485; OEM PN (none) -> RC0402JR-070RL
- R7: value 5.1k -> 1k; MPN RC0402FR-075K1L -> C106235; OEM PN (none) -> RC0402FR-071KL
- R8: MPN RC0402FR-071KL -> C106235; OEM PN (none) -> RC0402FR-071KL
- SW1: renamed from SW3; MPN SN74LVC1G3157DCKR -> C38663; OEM PN (none) -> SN74LVC1G3157DCKR
- SW3: renamed from SW1; MPN TS-1088R-02026 -> C455280; OEM PN (none) -> TS-1088R-02026
- SW4: renamed from SW2; MPN TS-1088R-02026 -> C455280; OEM PN (none) -> TS-1088R-02026
- U1: renamed from U2; MPN BGA2818,115 -> None; Note (none) -> Not available from LCSC.; OEM PN (none) -> BGA2818,115
- U5: renamed from U3; MPN MCP6566T-E/LT -> C623508; Note (none) -> Out of stock at LCSC.; OEM PN (none) -> MCP6566T-E/LT
- U7: renamed from U5; MPN W25Q128JVSIQ -> C97521; OEM PN (none) -> W25Q128JVSIQ
- U8: renamed from U6; MPN RP2040 -> C2040; OEM PN (none) -> RP2040
- X1: MPN SF2321D -> C3283372; Note (none) -> Out of stock at LCSC.; OEM PN (none) -> SF2321D
- Y1: MPN TAXM12M4RKDCDT2T -> C403945; OEM PN (none) -> TAXM12M4RKDCDT2T
- renumbered TP3 to TP1, TP5 to TP10, TP7 to TP11, TP1 to TP2, TP6 to TP4, TP2 to TP5, TP4 to TP9
Connections:
- net +3V3: now also C26.2, J3.2 (Pin_2), R3.1, C13.2, C14.2, C32.1, C6.1, F1.1, F2.1, R11.1, R12.1, R16.1, R17.1, R2.1, R22.1, SW2.5 (VCC), U10.2 (VO), U3.8 (V+), U4.1 (VDD), U6.1 (E0), U6.8 (VCC), U9.3 (3V3); no longer C15.2, L1.2, R5.2
- net +5V: now also D6.1 (K), U10.3 (VI); no longer J3.1 (Pin_1)
- net DECODE: now also SW2.6 (S); no longer J3.5 (Pin_5)
- net GND: now also C15.1, C26.1, J3.4 (Pin_4), C10.1, C13.1, C14.1, C32.2, C4.2, C6.2, J2.A1 (GND), J2.A12 (GND), J2.B1 (GND), J2.B12 (GND), J5.5 (Pin_5), J6.11 (Pin_11), J6.2 (Pin_2), R10.2, R23.2, R8.2, R9.2, SW2.2 (GND), U10.1 (GND), U2.5 (PWDN), U2.6 (COMM), U3.4 (V-), U4.2 (VSS), U6.2 (E1), U6.3 (E2), U6.4 (VSS), U9.1 (GND), U9.11 (GND), U9.14 (GND), U9.2 (GND), U9.36 (GND), U9.37 (GND), U9.38 (GND), U9.39 (GND), U9.40 (GND), U9.41 (GND), U9.42 (GND), U9.43 (GND), U9.44 (GND), U9.45 (GND), U9.46 (GND), U9.47 (GND), U9.48 (GND), U9.49 (GND), U9.50 (GND), U9.51 (GND), U9.52 (GND), U9.53 (GND); no longer C26.2, J3.2 (Pin_2), J3.6 (Pin_6)
- net GNDPWR: now also J2.S1 (SHIELD)
- net MTL_BIAS: now also U5.4 (-); no longer U5.3 (+)
- net RF_DET_OUT: now also R5.2, TP3.1, U2.8 (VOUT), U3.3 (+); no longer TP5.1, U5.4 (-)
- net RSSI_HOLD: now also C15.2, SW2.4 (A); no longer C15.1, D2.2 (A)
- net USB_D+: now also J2.A6 (D+), J2.B6 (D+)
- net USB_D-: now also J2.A7 (D-), J2.B7 (D-)
- net VBUS: now also J2.A4 (VBUS), J2.A9 (VBUS), J2.B4 (VBUS), J2.B9 (VBUS)
- net at R3.2: now also C4.1, U2.4 (VPOS)
- net at R7.1: now also U3.2 (-), U4.6 (W)
- net RSSI_PEAK: now reaches D2.1 (K)
- net RSSI_PEAK: now also SW2.1 (B2), U3.6 (-)
- net ESP32_SPI_MISO: now reaches U8.12 (GPIO9)
- net ESP32_SPI_MISO: now also U9.19 (MTDI/GPIO12/ADC2_CH5)
- net ESP32_SPI_CS: now reaches U8.13 (GPIO10)
- net ESP32_SPI_CS: now also U9.21 (MTDO/GPIO15/ADC2_CH3)
- net ESP32_GPIO0_BOOT: now reaches U8.14 (GPIO11)
- net ESP32_GPIO0_BOOT: now also J3.6 (Pin_6), R22.2, U9.23 (GPIO0/BOOT/ADC2_CH1)
- net I2C0_SDA: now reaches U8.15 (GPIO12)
- net I2C0_SDA: now also J6.6 (Pin_6), R16.2
- net I2C0_SCL: now reaches U8.16 (GPIO13)
- net I2C0_SCL: now also J6.7 (Pin_7), R17.2
- net ESP32_ENABLE: now reaches U8.17 (GPIO14)
- net ESP32_ENABLE: now also J3.1 (Pin_1), R18.1, R23.1
- net GNSS_UART0_TX: now reaches U8.2 (GPIO0)
- net GNSS_UART0_TX: now also J5.2 (Pin_2)
- net ESP32_UART0_TX: now reaches U8.27 (GPIO16)
- net ESP32_UART0_TX: now also J3.5 (Pin_5), R20.2
- net ESP32_UART0_RX: now reaches U8.28 (GPIO17)
- net ESP32_UART0_RX: now also J3.3 (Pin_3), R19.2
- net AUX_GPIOA: now reaches U8.29 (GPIO18)
- net AUX_GPIOA: now also J6.8 (Pin_8)
- net GNSS_UART0_RX: now reaches U8.3 (GPIO1)
- net GNSS_UART0_RX: now also J5.3 (Pin_3)
- net AUX_GPIOB: now reaches U8.35 (GPIO23)
- net AUX_GPIOB: now also J6.9 (Pin_9)
- net I2C1_SDA: now reaches U8.4 (GPIO2)
- net I2C1_SDA: now also R11.2, TP7.1, U4.4 (SDA), U6.5 (SDA)
- net AUX_GPIOC: now reaches U8.41 (GPIO29_ADC3)
- net AUX_GPIOC: now also J6.10 (Pin_10)
- net I2C1_SCL: now reaches U8.5 (GPIO3)
- net I2C1_SCL: now also R12.2, TP6.1, U4.3 (SCL), U6.6 (SCL)
- net GNSS_PPS: now reaches U8.8 (GPIO6)
- net GNSS_PPS: now also J5.4 (Pin_4)
- net ESP32_SPI_CLK: now reaches U8.9 (GPIO7)
- net ESP32_SPI_CLK: now also U9.18 (MTMS/GPIO14/ADC2_CH6)
- removed net 3V3_FILT_RF_DET: C3.2, L1.1, R3.1
- net RF_DET_IN: no longer names the net of U1.3
- net RF_DET_IN: now also C9.1; no longer C26.1
- net UART_RX renamed UART1_RX
- net UART1_RX: now also J6.4 (Pin_4); no longer J3.4 (Pin_4)
- net UART_TX renamed UART1_TX
- net UART1_TX: now also J6.3 (Pin_3); no longer J3.3 (Pin_3)
- net ~{RSSI_CLEAR}: no longer names the net of R5.1
- net ~{RSSI_CLEAR}: now also U2.7 (VSET); no longer U8.11 (GPIO8)
- new net: D2.2 (A), U3.7
- new net: R20.1, U9.30 (U0RXD/GPIO3)
- new net: R19.1, U9.31 (U0TXD/GPIO1)
- new net: D6.2 (A), J6.1 (Pin_1)
- new net: F2.2, J6.5 (Pin_5)
- new net: R18.2, U9.8 (EN/CHIP_PU)
- new net: J2.A5 (CC1), R9.1
- new net: J2.B5 (CC2), R10.1
- new net: C3.2, R2.2, U2.1 (VPOS)
- new net: F1.2, J5.1 (Pin_1)
- new net ESP32_SPI_MOSI: U8.11 (GPIO8), U9.20 (MTCK/GPIO13/ADC2_CH4)
- new net RF_DET_IN+: C9.2, L1.1, U2.2 (INHI)
- new net RF_DET_IN-: C10.2, L1.2, U2.3 (INLO)
- new net RF_LEVEL: TP5.1, U3.1, U3.5 (+), U4.5 (B), U5.3 (+)
- new net RSSI_DSCHRG: R8.1, SW2.3 (B1)
- no-connect marks 20 -> 26
Other:
- note added: "100k Digital Potentiometer for Adjustable Gain A_min = 0 A_max = 101"
- note added: "2kB EEPROM"
- note added: "Analog switch I_max = 128mA"
- note added: "Comparator Specs Propagation Delay ~50ns Fall Time 20ns"
- note added: "Discharge RC Time Constant T = 44ns 95% discharged = 132ns"
- note added: "ESP32 Pico Mini 02/02U 802.11 and Bluetooth Module"
- note added: "ESPFlash 2x3 Programming Header"
- note added: "Enabled during decode interval to sample RSSI of packet."
- note added: "For firmware update and logging only."
- note added: "HSPI Interface Used for AT Commands"
- note added: "I2C Address 3x LSBs: 0b001"
- note added: "I_in,max = 200mA (conservative guess, heavily dependent on GPIO)"
- note added: "I_in_max = 368mA 802.11b, 20 MHz, 1 Mbps, @19.5dBm"
- note added: "Ideal Peak Detector"
- note added: "Keep capacitance on V_OUT low! I_out,max = 400uA."
- note added: "NOTE: TX/RX nets refer to pins on host, not ESP32!"
- note added: "RSSI Hold and Discharge"
- note added: "TODO: add pmos polarity protection on 3.3V, make single row, add i2c pins"
- note added: "TX/RX swap happens here."
- note added: "USB C Connector"
- note added: "Use JSMSEMI or similar."
- note removed: "AD8314 has internal coupling cap, no external AC coupling required."
- note removed: "BW_video = 1 / (2*pi*13kOhms*(3.5pF+C_F)) Leave video bandwidth DNP to capture 1MHz modulation."
- note removed: "Enabled during decode interval to sample RSSI of packet. Enable Time: 1.5us Disable Time: 50ns"
- note removed: "Micro USB Connector"
- note removed: "V_DN descends from 2.25V to GND proportional to log of input RF power."
- note removed: "Waveform averaging timing cap"
- note removed: "f_c = 1.59MHz"
- moved on the sheet: C1, C15, C16, C17, C18, C19, C2, C20, C21, C22, C23, C24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

Commit message: Add Rev D PCBA files
Parts:
- removed C7, C8: 39pF, Capacitor_SMD:C_0402_1005Metric, symbol Device:C
- removed U1: BGA2818, Package_TO_SOT_SMD:SOT-363_SC-70-6, symbol RF_Amplifier:BGA2818
- added C33: 22nF, Capacitor_SMD:C_0402_1005Metric, symbol Device:C
- added C34: 10uF, Capacitor_SMD:C_0805_2012Metric, symbol Device:C
- added C35, C36: 100pF, Capacitor_SMD:C_0402_1005Metric, symbol Device:C
- added C37, C38: 12pF, Capacitor_SMD:C_0402_1005Metric, symbol Device:C
- added C39: 0.1uF, Capacitor_SMD:C_0402_1005Metric, symbol Device:C
- added D7: ORANGE, LED_SMD:LED_0603_1608Metric, symbol Device:LED
- added L2: 27nH RF, Inductor_SMD:L_0402_1005Metric, symbol Device:L
- added L3: 82nH RF, Inductor_SMD:L_0402_1005Metric, symbol Device:L
- added R28: 1k, Resistor_SMD:R_0402_1005Metric, symbol Device:R_US
- added R29: 20R, Resistor_SMD:R_0402_1005Metric, symbol Device:R_US
- added R30: 750R, Resistor_SMD:R_0402_1005Metric, symbol Device:R_US
- added R31: 6.8k, Resistor_SMD:R_0402_1005Metric, symbol Device:R_US
- added R32: 0R, Resistor_SMD:R_0402_1005Metric, symbol Device:R_US
- added U11: BLB01, Custom_Package_DFN_QFN:DFN-8-1EP_2x2mm_P0.5mm_EP0.9x1.5mm, symbol Custom_RF_Amplifier:BLB01
- C2: value 22nF -> 100pF; MPN C107026 -> C106200; OEM PN CC0402KRX7R9BB223 -> CC0402JRNPO9BN101
- F1, F2: OEM PN BSMD0402L-020 -> BSMD0402L-020
- J5: value Conn_01x05_Pin -> 1x5 2.54mm Pin Header; now not fitted
- J6: value Conn_01x11_Pin -> 1x11 2.54mm Pin Header; now not fitted
- L1: MPN C361505 -> C361505; OEM PN SDWL1005C8N2JSTF -> SDWL1005C8N2JSTF
- PCB1: REV REV C -> REV D
- X1: value SF2321D -> TA2003A; footprint Custom_Filter:Filter_SAW-6_3.8x3.8mm -> Custom_Filter:Filter_SAW-6_3.0x3.0mm; MPN C3283372 -> (none); OEM PN SF2321D -> TA2003A; Standard Cost 1.10 -> 2.50
Connections:
- net +3V3: now also C33.2, C39.1, R31.1, R32.1; no longer C2.1
- net GND: now also C36.2, C37.1, C39.2, R28.2, R30.2, U11.9 (G); no longer C2.2
- net RF_DET_OUT: now also C34.1; no longer U3.3 (+)
- net RF_IN: now also C2.1
- net RF_LNA_IN: now also C35.2, L2.2, U11.2
- net RF_SAW_IN: now also C2.2
- net RF_SAW_OUT: now also C35.1
- net RSSI_PEAK: now also R29.1; no longer SW2.1 (B2)
- net ~{RESET}: now also C33.1
- net ESP_LED: now reaches U9.29 (GPIO5)
- net ESP_LED: now also D7.2 (A)
- net RF_LNA_OUT: now reaches C9.1
- net RF_LNA_OUT: now also C38.2
- net MTL_BIAS renamed TL_BIAS
- net MTL_HI_BIAS renamed TL_LO_BIAS
- net MTL_HI_PWM renamed TL_LO_PWM
- net MTL_LO_BIAS renamed TL_HI_BIAS
- net MTL_LO_PWM renamed TL_HI_PWM
- new net: C36.1, L3.1, R32.2
- new net: C37.2, L2.1, R31.2, U11.1 (Vcc)
- new net: D7.1 (K), R30.1
- new net: R29.2, SW2.1 (B2)
- new net RF_DET_OUT_FILT: C34.2, R28.1, U3.3 (+)
- new net RF_LNA_OUT': C38.1, L3.2, U11.7
- no-connect marks 26 -> 25
Other:
- note added: "GNSS Header"
- note added: "GPIO Header"
- note added: "Keep capacitance on VOUT low! I_out,max = 400uA."
- note added: "RF Input Signal Chain"
- note added: "Variable Gain Op-Amp"
- note removed: "+30dB Gain"
- note removed: "Keep capacitance on V_OUT low! I_out,max = 400uA."
- note removed: "LNA"
- note removed: "LNA Requirements: AC coupling caps must be <100pF. 22nF decoupling cap must be close to IC. Use multiple vias for ground."
- note removed: "RF Signal Chain"
- note removed: "TODO: add pmos polarity protection on 3.3V, make single row, add i2c pins"
- moved on the sheet: C1, C10, C13, C14, C15, C16, C17, C18, C19, C2, C20, C21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

Commit message: Update Rev D fab files
Parts:
- renumbered C39 to C1, C35 to C10, C38 to C11, C10 to C12, C31 to C14, C32 to C15, C6 to C2, C16 to C20, C17 to C21, C18 to C22, C19 to C23, C20 to C24, C21 to C25, C22 to C26, C23 to C27, C24 to C28, C25 to C29, C26 to C30, C14 to C31, C27 to C32, C15 to C33, C28 to C34, C29 to C35, C33 to C36, C30 to C37, C37 to C5, C36 to C6, C9 to C7, C34 to C8, C2 to C9, D3 to D2, D4 to D3, D5 to D4, D7 to D5, D2 to D6, D6 to D7, J6 to J5, J5 to J6, L2 to L1, L3 to L2, L1 to L3, R2 to R1, R9 to R10, R10 to R11, R26 to R13, R27 to R14, R30 to R15, R11 to R16, R12 to R17, R13 to R18, R14 to R19, R3 to R2, R15 to R20, R16 to R21, R17 to R22, R29 to R23, R21 to R24, R8 to R25, R24 to R26, R25 to R27, R18 to R28, R19 to R29, R31 to R3, R20 to R30, R22 to R31, R23 to R32, R32 to R4, R28 to R5, R5 to R6, R1 to R8, R4 to R9, TP3 to TP1, TP6 to TP2, TP7 to TP3, TP1 to TP4, TP2 to TP5, TP4 to TP6, TP5 to TP7, U3 to U1, U9 to U10, U11 to U2, U2 to U3, U10 to U5, U5 to U6, U6 to U7, U7 to U8, U8 to U9
