File: kicad/proto_data_slicer_board/proto_data_slicer_board.kicad_sch (KiCad schematic)
At the start: 18 parts, among them U1 MCP6566

Commit message: Add data slicer and LNA proto boards
Parts:
- R2: value 2M -> 100k
Connections:
- net +3V3: no longer R2.1
- new net TL_BIAS: R2.1
Changed lines of the file:
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@@
-	(wire
-		(pts
-			(xy 97.79 66.04) (xy 97.79 67.31)
-		)
-		(stroke
-			(width 0)
-			(type default)
-		)
-	)
 	(wire
 		(pts
@@
 	(wire
 		(pts
+			(xy 97.79 63.5) (xy 97.79 67.31)
+		)
+		(stroke
+			(width 0)
+			(type default)
+		)
+	)
+	(wire
+		(pts
 			(xy 161.29 59.69) (xy 161.29 81.28)
 		)
@@
 		(pts
 			(xy 138.43 59.69) (xy 147.32 59.69)
+		)
+		(stroke
+			(width 0)
+			(type default)
+		)
+	)
+	(wire
+		(pts
+			(xy 105.41 63.5) (xy 97.79 63.5)
 		)
 		(stroke
@@
 			)
 			(justify left bottom)
+		)
+	)
+	(label "TL_BIAS"
+		(at 105.41 63.5 180)
+		(fields_autoplaced yes)
+		(effects
+			(font
+				(size 1.27 1.27)
+			)
+			(justify right bottom)
 		)
 	)
@@
 	)
 	(symbol
-		(lib_id "power:+3V3")
-		(at 97.79 66.04 0)
-		(unit 1)
-		(exclude_from_sim no)
-		(in_bom yes)
-		(on_board yes)
-		(dnp no)
-		(fields_autoplaced yes)
-		(property "Reference" "#PWR01"
-			(at 97.79 69.85 0)
-			(effects
-				(font
-					(size 1.27 1.27)
-				)
-				(hide yes)
-			)
-		)
-		(property "Value" "+3V3"
-			(at 97.79 60.96 0)
-			(effects
-				(font
-					(size 1.27 1.27)
-				)
-			)
-		)
-		(property "Footprint" ""
-			(at 97.79 66.04 0)
-			(effects
-				(font
-					(size 1.27 1.27)
-				)
-				(hide yes)
-			)
-		)
-		(property "Datasheet" ""
-			(at 97.79 66.04 0)
-			(effects
-				(font
-					(size 1.27 1.27)
-				)
-				(hide yes)
-			)
-		)
-		(property "Description" "Power symbol creates a global label with name \"+3V3\""
-			(at 97.79 66.04 0)
-			(effects
-				(font
-					(size 1.27 1.27)
-				)
-				(hide yes)
-			)
-		)
-		(pin "1"
-		)
-		(instances
-			(project ""
-				(path "/49d83cd2-f051-4cc2-a9c8-fdc67599e457"
-					(reference "#PWR01")
-					(unit 1)
-				)
-			)
-		)
-	)
-	(symbol
 		(lib_id "power:GND")
 		(at 97.79 118.11 0)
@@
 			)
 		)
-		(property "Value" "2M"
+		(property "Value" "100k"
 			(at 95.25 72.3899 0)
 			(effects
